File: PCB Design/ESP_Bare_v2.brd (EAGLE design)
At the start: 91.5 x 46.5 mm, 69 parts, among them Q1 NPN_S8050, Q2 NPN_S8050, Q3 BC848 30V 100mA, Q4 BSS138

Commit message: Fix issues
• Fix WIFI button routing
• Fix Photo-Resistor routing
Parts:
- moved C7 12.3 mm to (34.9, 50.9), turned to 0 degrees
Connections:
- net 3.3V: no longer R21.2
- net A0: now also R21.2
- net GND: now also YD-3414.1
- net RX: now also YD-3414.4; no longer YD-3414.1
Routing:
- net 3.3V: track 285.5 -> 283.5 mm
- net IO14: track 46.3 -> 48.2 mm
- net A0: track 62.3 -> 63.9 mm
- net GND: vias 60 -> 61
