File: PCB Design/ESP_Bare_v2.sch (EAGLE design)
At the start: 69 parts, among them Q1 NPN_S8050, Q2 NPN_S8050, Q3 BC848 30V 100mA, Q4 BSS138

Commit message: Fix issues
• Fix WIFI button routing
• Fix Photo-Resistor routing
Connections:
- net 3.3V: no longer R21.2
- net A0: now also R21.2
- net GND: now also YD-3414.3
- net RX: now also YD-3414.2; no longer YD-3414.3
Changed lines of the file:
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@@
 <text x="99.06" y="-10.16" size="1.778" layer="91" rot="R270">NPN_S8050</text>
 <text x="99.06" y="-30.48" size="1.778" layer="91" rot="R270">NPN_S8050</text>
-<text x="195.58" y="0" size="1.778" layer="91">WiFi ON/OFF</text>
+<text x="190.5" y="5.08" size="1.778" layer="91">WiFi ON/OFF</text>
 <text x="195.58" y="-15.24" size="1.778" layer="91">WiFi State LED</text>
 <text x="195.58" y="-35.56" size="1.778" layer="91">Alarm State LED</text>
@@
 <attribute name="NAME" x="-9.144" y="128.778" size="1.524" layer="95"/>
 </instance>
-<instance part="GND9" gate="1" x="185.42" y="-5.08" smashed="yes" rot="R270">
-<attribute name="VALUE" x="182.88" y="-2.54" size="1.778" layer="96" rot="R270"/>
+<instance part="GND9" gate="1" x="185.42" y="2.54" smashed="yes" rot="R270">
+<attribute name="VALUE" x="182.88" y="5.08" size="1.778" layer="96" rot="R270"/>
 </instance>
 <instance part="D2" gate="G$1" x="205.74" y="-22.86" smashed="yes" rot="R270">
@@
 <segment>
 <pinref part="PH1" gate="G$1" pin="2"/>
-<wire x1="256.54" y1="180.34" x2="256.54" y2="177.8" width="0.1524" layer="91"/>
 <label x="256.54" y="162.56" size="1.778" layer="95" rot="R270" xref="yes"/>
-<wire x1="256.54" y1="177.8" x2="256.54" y2="162.56" width="0.1524" layer="91"/>
-<wire x1="256.54" y1="177.8" x2="248.92" y2="177.8" width="0.1524" layer="91"/>
-<junction x="256.54" y="177.8"/>
-<pinref part="R21" gate="G$1" pin="2"/>
-<wire x1="248.92" y1="172.72" x2="248.92" y2="177.8" width="0.1524" layer="91"/>
+<wire x1="256.54" y1="180.34" x2="256.54" y2="162.56" width="0.1524" layer="91"/>
 </segment>
 <segment>
@@
 </segment>
 <segment>
-<wire x1="195.58" y1="-5.08" x2="187.96" y2="-5.08" width="0.1524" layer="91"/>
 <pinref part="GND9" gate="1" pin="GND"/>
-<wire x1="195.58" y1="-5.08" x2="195.58" y2="-2.54" width="0.1524" layer="91"/>
-<wire x1="195.58" y1="-2.54" x2="208.28" y2="2.54" width="0.1524" layer="91"/>
+<wire x1="187.96" y1="2.54" x2="208.28" y2="2.54" width="0.1524" layer="91"/>
 <pinref part="YD-3414" gate="G$1" pin="1"/>
 </segment>
@@
 <wire x1="266.7" y1="165.1" x2="266.7" y2="157.48" width="0.1524" layer="91"/>
 <label x="266.7" y="157.48" size="1.778" layer="95" rot="R270" xref="yes"/>
+</segment>
+<segment>
+<pinref part="YD-3414" gate="G$1" pin="3"/>
+<wire x1="218.44" y1="2.54" x2="223.52" y2="2.54" width="0.1524" layer="91"/>
+<label x="223.52" y="2.54" size="1.778" layer="95" xref="yes"/>
 </segment>
 </net>
@@
 </segment>
 <segment>
-<wire x1="236.22" y1="-5.08" x2="231.14" y2="-5.08" width="0.1524" layer="91"/>
 <label x="236.22" y="-5.08" size="1.778" layer="95" xref="yes"/>
-<wire x1="218.44" y1="2.54" x2="231.14" y2="-2.54" width="0.1524" layer="91"/>
-<wire x1="231.14" y1="-2.54" x2="231.14" y2="-5.08" width="0.1524" layer="91"/>
-<pinref part="YD-3414" gate="G$1" pin="3"/>
+<pinref part="YD-3414" gate="G$1" pin="2"/>
+<wire x1="228.6" y1="-5.08" x2="236.22" y2="-5.08" width="0.1524" layer="91"/>
+<wire x1="208.28" y1="-5.08" x2="205.74" y2="-5.08" width="0.1524" layer="91"/>
+<wire x1="205.74" y1="-5.08" x2="205.74" y2="-10.16" width="0.1524" layer="91"/>
+<wire x1="205.74" y1="-10.16" x2="228.6" y2="-10.16" width="0.1524" layer="91"/>
+<wire x1="228.6" y1="-10.16" x2="228.6" y2="-5.08" width="0.1524" layer="91"/>
 </segment>
 </net>
@@
 <wire x1="256.54" y1="190.5" x2="256.54" y2="193.04" width="0.1524" layer="91"/>
 <label x="256.54" y="193.04" size="1.778" layer="95" rot="R90" xref="yes"/>
-</segment>
-</net>
+<pinref part="R21" gate="G$1" pin="2"/>
+<wire x1="248.92" y1="172.72" x2="248.92" y2="190.5" width="0.1524" layer="91"/>
+<wire x1="248.92" y1="190.5" x2="256.54" y2="190.5" width="0.1524" layer="91"/>
+<junction x="256.54" y="190.5"/>
+</segment>
+</net>
