File: PCB Design/ESP_Bare_v3.1.brd (EAGLE design)
At the start: 91.5 x 46.5 mm, 69 parts, among them Q1 NPN_S8050, Q2 NPN_S8050, Q3 BC848 30V 100mA, Q4 BSS138

Commit message: UPDATES
• Final Clock PCP
• ATtiny code: some changes
• ESP code: more work done
Parts:
- removed R22: 10k, rcl:R0603
- removed S2, S3, S4: (no value), switch-omron:B3F-10XX
- added Q5: IRLML6344, IRLML6344:SOT23
- added R25: 18k, resistor:R0603
- added S5, S6, S7: MOMENTARY-SWITCH-SPST-SMD-4.6X2.8MM, SparkFun-Switches:TACTILE_SWITCH_SMD_4.6X2.8MM
- added SG, SP: TPB1,27, testpad:B1,27
- C7: value 10uf -> 100nf
- D5: value 1A/23V/620mV -> 1A/23V/620mV BAT20JFILM
- R18: value 470R -> 470
- moved R23 4.02 mm to (84.1, 53.1)
- moved YD-3414 0.13 mm to (58.2, 34.0)
Connections:
- removed net BAT: CR1220.+$1, DS3231.14, R23.2
- new net A1: ATTINY841.12, R23.1
- new net RTC_BAT: CR1220.+$1, DS3231.14, Q5.3
- net 5V: now also Q5.1, R25.2
- net GND: now also R25.1, S5.1, S5.2, S6.1, S6.2, S7.1, S7.2, SG.TP; no longer R22.1, S2.3, S3.3, S4.3
- net IO0: now also S6.3, S6.4; no longer S3.2
- net IO12: now also S5.3, S5.4; no longer S2.2
- net IO13: now also SP.TP
- net IO2: now also S7.3, S7.4; no longer S4.2
- net N$5: now also Q5.2, R23.2; no longer ATTINY841.12, R22.2, R23.1
Routing:
- net RTC_BAT: track 0.00 -> 43.2 mm, vias 0 -> 2
- net BAT: track 40.8 -> 0.00 mm, vias 2 -> 0
- net IO0: track 39.6 -> 51.0 mm, vias 0 -> 2
- net IO12: track 23.6 -> 33.8 mm, vias 0 -> 2
- net IO2: track 61.1 -> 67.6 mm
- net A1: track 0.00 -> 5.92 mm
- net IO13: track 38.1 -> 42.2 mm
- net N$5: track 5.75 -> 3.12 mm
- net IO4: track 153.6 -> 155.8 mm
- net 5V: track 144.5 -> 146.5 mm
- net RX: track 85.0 -> 86.2 mm
- net A2: track 14.2 -> 15.3 mm
- net IO5: track 194.6 -> 195.3 mm
- net GND: track 20.6 -> 20.7 mm, vias 61 -> 60
Other:
- outline, holes or cut-outs redrawn
- board text added: "BY ALBERT KRAVCOV REV2"
- board text removed: "BY ALBERT KRAVCOV REV1"
