File: PCB Design/ESP_Bare_v3.1.sch (EAGLE design)
At the start: 69 parts, among them Q1 NPN_S8050, Q2 NPN_S8050, Q3 BC848 30V 100mA, Q4 BSS138

Commit message: UPDATES
• Final Clock PCP
• ATtiny code: some changes
• ESP code: more work done
Parts:
- removed R22: 10k, rcl:R-EU_R0603
- removed S2, S3, S4: (no value), switch-omron:10-XX
- added Q5: IRLML6344, IRLML6344:IRLML6344
- added R25: 18k, resistor:R-EU_R0603
- added S5, S6, S7: MOMENTARY-SWITCH-SPST-SMD-4.6X2.8MM, SparkFun-Switches:MOMENTARY-SWITCH-SPST-SMD-4.6X2.8MM
- added SG, SP: TPB1,27, testpad:TPB1,27
- C7: value 10uf -> 100nf
- D5: value 1A/23V/620mV -> 1A/23V/620mV BAT20JFILM
- R18: value 470R -> 470
Connections:
- removed net BAT: CR1220.+, DS3231.VBAT, R23.2
- new net A1: ATTINY841.PA1, R23.1
- new net RTC_BAT: CR1220.+, DS3231.VBAT, Q5.D
- net 5V: now also Q5.G, R25.2
- net GND: now also R25.1, S5.1, S6.1, S7.1, SG.TP; no longer R22.1, S2.P, S3.P, S4.P
- net IO0: now also S6.2; no longer S3.S1
- net IO12: now also S5.2; no longer S2.S1
- net IO13: now also SP.TP
- net IO2: now also S7.2; no longer S4.S1
- net N$5: now also Q5.S, R23.2; no longer ATTINY841.PA1, R22.2, R23.1
Other:
- note added: "BATTERY HOLDER"
- note added: "FLASH POGO"
- moved on the sheet: ATTINY841, C10, C9, CR1220, D5, D6, DS3231, FL01, FL02, LS1, PH1, Q3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
